Commit message: 25_11_2023_latenight

File: description/robot_core.xacro (robot description, xacro)
@@ -1,4 +1,5 @@
 <?xml version="1.0"?>
 <robot xmlns:xacro="http://www.ros.org/wiki/xacro"  name="robot">
+    <xacro:include filename="inertias.xacro"/>
     <material name= "white">
         <color rgba="1 1 1 1"/>
@@ -29,4 +30,13 @@
            <material name="white" />
         </visual>
+        <collision>
+            <origin xyz="0.15 0.0 0.075" rpy="0.0 0.0 0.0"/>
+            <geometry>
+                <box size=" 0.3 0.3 0.15 "/>
+            </geometry>
+        </collision>
+    <xacro:inertial_box mass= "0.5" x="0.3" y="0.3" z= "0.15">
+        <origin xyz="0.15 0.0 0.075" rpy="0.0 0.0 0.0"/>
+     </xacro:inertial_box>
     </link>
     <!-- left wheel link-->
@@ -44,4 +54,12 @@
            <material name="black" />
         </visual>
+        <collision>
+            <geometry>
+                <cylinder radius=".05" length="0.04"/>
+            </geometry>
+        </collision>
+        <xacro:inertial_cylinder mass= "0.1" length="0.04" radius="0.05">
+            <origin xyz="0.0 0.0 0.0" rpy="0.0 0.0 0.0"/>
+        </xacro:inertial_cylinder>
     </link>
     <!-- right wheel link-->
@@ -59,4 +77,12 @@
            <material name="black" />
         </visual>
+        <collision>
+            <geometry>
+                <cylinder radius=".05" length="0.04"/>
+            </geometry>
+        </collision>
+        <xacro:inertial_cylinder mass= "0.1" length="0.04" radius="0.05">
+            <origin xyz="0.0 0.0 0.0" rpy="0.0 0.0 0.0"/>
+        </xacro:inertial_cylinder>
     </link>
      <!-- castor wheel link-->
@@ -73,4 +99,12 @@
            <material name="blue" />
         </visual>
+        <collision>
+                <geometry>
+                    <sphere radius="0.05"/>
+                </geometry>
+        </collision>
+        <xacro:inertial_sphere mass= "0.1" radius="0.05">
+            <origin xyz="0.0 0.0 0.0" rpy="0.0 0.0 0.0"/>
+        </xacro:inertial_sphere>
     </link>
 </robot>
