Commit message: update_with_world creation and gazebo_control.xacro

File: description/robot.urdf.xacro (robot description, xacro)
@@ -2,3 +2,4 @@
 <robot xmlns:xacro="http://www.ros.org/wiki/xacro"  name="robot">
     <xacro:include filename="robot_core.xacro" />
+     <xacro:include filename="gazebo_control.xacro" />
 </robot>

File: description/robot_core.xacro (robot description, xacro)
@@ -40,4 +40,7 @@
      </xacro:inertial_box>
     </link>
+    <gazebo reference = "chassis">
+        <material>Gazebo/white</material>
+    </gazebo>
     <!-- left wheel link-->
     <joint name="left_wheel_joint" type="continuous">
@@ -63,4 +66,7 @@
         </xacro:inertial_cylinder>
     </link>
+    <gazebo reference = "left_wheel">
+        <material>Gazebo/Black</material>
+    </gazebo>
     <!-- right wheel link-->
     <joint name="right_wheel_joint" type="continuous">
@@ -86,4 +92,7 @@
         </xacro:inertial_cylinder>
     </link>
+    <gazebo reference = "right_wheel">
+        <material>Gazebo/Black</material>
+    </gazebo>
      <!-- castor wheel link-->
      <joint name="castor_wheel_joint" type="fixed">
@@ -108,3 +117,8 @@
         </xacro:inertial_sphere>
     </link>
+    <gazebo reference = "castor_wheel">
+        <material>Gazebo/Blue</material>
+        <mu1 value="0.001"/>
+        <mu2 value="0.001"></mu2>
+    </gazebo>
 </robot>
